File: hw_pcb/mbadge25_v1/mbadge25.kicad_sch (KiCad schematic)
At the start: 25 parts, among them J1 USB4105-GF-A, J2 BAT, J3 OLED_I2C, T1 LP0404N3T5G, U1 ESP32-C3-MINI-1, U2 XC6220B331MR

Commit message: v1 draft PCB layout
Parts:
- added D2: WS2812B, Library_FP_mbadge25:LED_WS2812B_PLCC4_5.0x5.0mm_P3.2mm, symbol Library_SYM_mbadge25:WS2812B
- added J4: BAT, Library_FP_mbadge25:Pad_6.0mm_Drill3.0mm, symbol Library_SYM_mbadge25:Conn_01x01
- added J5: GND, Library_FP_mbadge25:Pad_6.0mm_Drill3.0mm, symbol Library_SYM_mbadge25:Conn_01x01
- added J6: BAT, Library_FP_mbadge25:Pad_1.2mm_Drill0.7mm, symbol Library_SYM_mbadge25:Conn_01x01
- added J7: GND, Library_FP_mbadge25:Pad_1.2mm_Drill0.7mm, symbol Library_SYM_mbadge25:Conn_01x01
- added R8: 220E, Library_FP_mbadge25:R_1206_3216Metric_Pad1.30x1.75mm, symbol Library_SYM_mbadge25:R
- C1, C2, C3, C7, C8, C9: footprint PCM_Capacitor_SMD_AKL:C_0805_2012Metric_Pad1.18x1.45mm_HandSolder -> Library_FP_mbadge25:C_1206_3216Metric_Pad1.33x1.80mm
- C4, C5, C6: footprint PCM_Capacitor_SMD_AKL:CP_Elec_6.3x5.9 -> Library_FP_mbadge25:C_1206_3216Metric_Pad1.33x1.80mm
- D1: footprint (none) -> Library_FP_mbadge25:D_SOD-523
- J2: footprint (none) -> Library_FP_mbadge25:PinHeader_1x02_P2.54mm_Vertical
- J3: footprint (none) -> Library_FP_mbadge25:OLED_128x32
- R1, R2, R3, R4, R5, R6, R7: footprint Resistor_SMD:R_0805_2012Metric -> Library_FP_mbadge25:R_1206_3216Metric_Pad1.30x1.75mm
- S1, S2: footprint Button_Switch_THT:SW_PUSH_6mm -> Library_FP_mbadge25:SW_SPST
- T1: footprint (none) -> Library_FP_mbadge25:SOT-23-3
- U1: footprint PCM_Espressif:ESP32-C3-MINI-1 -> Library_FP_mbadge25:ESP32-C3-MINI-1
- U2: footprint Package_TO_SOT_SMD:SOT-23-5 -> Library_FP_mbadge25:SOT-23-5_HandSoldering
Connections:
- net SCL is gone; now on net IO8.SCL: J3.2 (Pin_2)
- net SDA is gone; now on net IO7.SDA: J3.1 (Pin_1)
- net GND: now also S1.2, S2.2, D2.3 (VSS), J5.1 (Pin_1), J7.1 (Pin_1); no longer S1.3, S2.3
- net VBAT: now also J4.1 (Pin_1), J6.1 (Pin_1)
- net at C8.1 (+), R7.1 (+), U1.8 (EN/CHIP_PU): now also S2.1; no longer S2.4
- net 5V0: now reaches C4.1 (+), C5.1 (+), D1.1 (K-), T1.3 (S), U2.1 (VIN), U2.3 (CE)
- net 5V0: now also D2.1 (VDD)
- net IO9: now reaches C7.1 (+), R6.1 (+), U1.23 (GPIO9)
- net IO9: now also S1.1; no longer S1.4
- net IO10: now reaches U1.16 (GPIO10)
- net IO4: now reaches U1.18 (GPIO4/ADC1_CH4)
- net IO5: now reaches U1.19 (GPIO5/ADC2_CH0)
- net IO6.RGB: now reaches U1.20 (GPIO6)
- net IO6.RGB: now also R8.2 (-)
- net IO7.SDA: now reaches U1.21 (GPIO7)
- net IO8.SCL: now reaches U1.22 (GPIO8)
- net IO20.RX: now reaches U1.30 (GPIO20/U0RXD)
- net IO21.TX: now reaches U1.31 (GPIO21/U0TXD)
- net IO2: now reaches U1.5 (GPIO2/ADC1_CH2)
- net IO3: now reaches U1.6 (GPIO3/ADC1_CH3)
- net USB.N renamed IO18.USBN
- net USB.P renamed IO19.USBP
- net VBUS renamed VUSB
- new net RGB.DI: D2.4 (DIN), R8.1 (+)
- new net RGB.DO: D2.2 (DOUT)
Other:
- moved on the sheet: C1, C2, C3, C4, C5, C6, C7, C8, C9, D1, J1, J2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

Commit message: v2 draft PCB layout
Parts:
- added J10: Conn_IO20.RX, Library_FP_mbadge25:PinHeader_1x01_P1.27mm_Vertical, symbol Library_SYM_mbadge25:Conn_01x01_Pin
- added J11: Conn_IO19.USBP, Library_FP_mbadge25:PinHeader_1x01_P1.27mm_Vertical, symbol Library_SYM_mbadge25:Conn_01x01_Pin
- added J12: Conn_IO18.USBN, Library_FP_mbadge25:PinHeader_1x01_P1.27mm_Vertical, symbol Library_SYM_mbadge25:Conn_01x01_Pin
- added J13: Conn_IO2, Library_FP_mbadge25:PinHeader_1x01_P1.27mm_Vertical, symbol Library_SYM_mbadge25:Conn_01x01_Pin
- added J14: Conn_IO3, Library_FP_mbadge25:PinHeader_1x01_P1.27mm_Vertical, symbol Library_SYM_mbadge25:Conn_01x01_Pin
- added J15: Conn_IO4, Library_FP_mbadge25:PinHeader_1x01_P1.27mm_Vertical, symbol Library_SYM_mbadge25:Conn_01x01_Pin
- added J16: Conn_IO5, Library_FP_mbadge25:PinHeader_1x01_P1.27mm_Vertical, symbol Library_SYM_mbadge25:Conn_01x01_Pin
- added J17: Conn_IO6.RGB, Library_FP_mbadge25:PinHeader_1x01_P1.27mm_Vertical, symbol Library_SYM_mbadge25:Conn_01x01_Pin
- added J18: Conn_IO7.SDA, Library_FP_mbadge25:PinHeader_1x01_P1.27mm_Vertical, symbol Library_SYM_mbadge25:Conn_01x01_Pin
- added J19: Conn_IO8.SCL, Library_FP_mbadge25:PinHeader_1x01_P1.27mm_Vertical, symbol Library_SYM_mbadge25:Conn_01x01_Pin
- added J20: Conn_IO10, Library_FP_mbadge25:PinHeader_1x01_P1.27mm_Vertical, symbol Library_SYM_mbadge25:Conn_01x01_Pin
- added J21: Conn_IO00, Library_FP_mbadge25:PinHeader_1x01_P1.27mm_Vertical, symbol Library_SYM_mbadge25:Conn_01x01_Pin
- added J22: Conn_IO01, Library_FP_mbadge25:PinHeader_1x01_P1.27mm_Vertical, symbol Library_SYM_mbadge25:Conn_01x01_Pin
- added J8: USB-C_BO, Library_FP_mbadge25:USB_C_BO, symbol Library_SYM_mbadge25:Conn_01x08
- added J9: Conn_IO21.TX, Library_FP_mbadge25:PinHeader_1x01_P1.27mm_Vertical, symbol Library_SYM_mbadge25:Conn_01x01_Pin
- D2, R8: now not fitted; now left out of the parts list
Connections:
- net DN: now also J8.5 (Pin_5)
- net DP: now also J8.6 (Pin_6)
- net GND: now also J8.1 (Pin_1)
- net IO10: now also J20.1 (Pin_1)
- net IO18.USBN: now also J12.1 (Pin_1)
- net IO19.USBP: now also J11.1 (Pin_1)
- net IO2: now also J13.1 (Pin_1)
- net IO20.RX: now also J10.1 (Pin_1)
- net IO21.TX: now also J9.1 (Pin_1)
- net IO3: now also J14.1 (Pin_1)
- net IO4: now also J15.1 (Pin_1)
- net IO5: now also J16.1 (Pin_1)
- net IO6.RGB: now also J17.1 (Pin_1)
- net IO7.SDA: now also J18.1 (Pin_1)
- net IO8.SCL: now also J19.1 (Pin_1)
- net VUSB: now also J8.2 (Pin_2)
- net EN: now reaches C8.1 (+), R7.1 (+), S2.1, U1.8 (EN/CHIP_PU)
- net CC2: now reaches J1.B5 (CC2), R2.1 (+)
- net CC2: now also J8.8 (Pin_8)
- net at U1.12 (GPIO0/ADC1_CH0/XTAL_32K_P): now also J21.1 (Pin_1)
- net at U1.13 (GPIO1/ADC1_CH1/XTAL_32K_N): now also J22.1 (Pin_1)
- net CC1: now reaches J1.A5 (CC1), R1.1 (+)
- net CC1: now also J8.4 (Pin_4)
- net SBU1: now reaches J1.A8 (SBU1)
- net SBU1: now also J8.7 (Pin_7)
- net SBU2: now reaches J1.B8 (SBU2)
- net SBU2: now also J8.3 (Pin_3)
- net IO9 renamed IO9.SW
- no-connect marks 2 -> 0
Other:
- moved on the sheet: C1, C2, C3, C4, C5, C6, C7, C8, C9, D1, J1, J2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

Commit message: draft PCB layout WIP
Parts:
- removed J13: Conn_IO2, Library_FP_mbadge25:PinHeader_1x01_P1.27mm_Vertical, symbol Library_SYM_mbadge25:Conn_01x01_Pin
- removed J14: Conn_IO3, Library_FP_mbadge25:PinHeader_1x01_P1.27mm_Vertical, symbol Library_SYM_mbadge25:Conn_01x01_Pin
- added J23: RGB, Library_FP_mbadge25:PinSocket_1x03_P1.27mm_Vertical, symbol Library_SYM_mbadge25:Conn_01x03
- added J24: Simple_Addon_v2, Library_FP_mbadge25:PinSocket_2x03_P2.54mm_Vertical, symbol Library_SYM_mbadge25:Simple_Addon_v2
- D2, R8: now fitted; now in the parts list
- J10, J11, J12, J15, J16, J17, J18, J19, J20, J21, J22, J9: now left out of the parts list
- J4, J5, J6, J7: now not fitted; now left out of the parts list
Connections:
- net 3V3: now also J24.1 (VCC)
- net 5V0: now also J23.2 (Pin_2)
- net GND: now also J23.3 (Pin_3), J24.2 (GND)
- net IO2: now also J24.6 (GPIO2)
- net IO3: now also J24.5 (GPIO1)
- net IO7.SDA: now also J24.3 (SDA)
- net IO8.SCL: now also J24.4 (SCL)
- net RGB.DO: now also J23.1 (Pin_1)
Other:
- moved on the sheet: J3, J8

Commit message: changed PCB dims, rearranged components
Parts:
- removed J17: Conn_IO6.RGB, Library_FP_mbadge25:PinHeader_1x01_P1.27mm_Vertical, symbol Library_SYM_mbadge25:Conn_01x01_Pin
- removed J18: Conn_IO7.SDA, Library_FP_mbadge25:PinHeader_1x01_P1.27mm_Vertical, symbol Library_SYM_mbadge25:Conn_01x01_Pin
- removed J19: Conn_IO8.SCL, Library_FP_mbadge25:PinHeader_1x01_P1.27mm_Vertical, symbol Library_SYM_mbadge25:Conn_01x01_Pin
Connections:
- net IO2 renamed IO2.SAO
- net IO3 renamed IO3.SAO
Changed lines of the file:
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@@
 	(title_block
 		(title "mbadge25")
-		(date "2025-03-19")
+		(date "2025-03-20")
 		(rev "v1")
 		(company "MakerVille")
@@
 		)
 	)
-	(label "IO2"
+	(label "IO2.SAO"
 		(at 222.25 55.88 0)
 		(effects
@@
 		)
 	)
-	(label "IO2"
+	(label "IO2.SAO"
 		(at 121.92 151.13 180)
 		(effects
@@
 		)
 	)
-	(label "IO3"
+	(label "IO3.SAO"
 		(at 121.92 153.67 180)
 		(effects
@@
 		)
 	)
-	(label "IO3"
+	(label "IO3.SAO"
 		(at 273.05 55.88 180)
 		(effects
@@
 	)
 	(symbol
-		(lib_id "Library_SYM_mbadge25:Conn_01x01_Pin")
-		(at 127 166.37 180)
-		(unit 1)
-		(exclude_from_sim no)
-		(in_bom no)
-		(on_board yes)
-		(dnp no)
-		(property "Reference" "J19"
-			(at 128.778 166.37 0)
-			(effects
-				(font
-					(size 1.27 1.27)
-				)
-			)
-		)
-		(property "Value" "Conn_IO8.SCL"
-			(at 126.365 163.83 0)
-			(effects
-				(font
-					(size 1.27 1.27)
-				)
-				(hide yes)
-			)
-		)
-		(property "Footprint" "Library_FP_mbadge25:PinHeader_1x01_P1.27mm_Vertical"
-			(at 127 166.37 0)
-			(effects
-				(font
-					(size 1.27 1.27)
-				)
-				(hide yes)
-			)
-		)
-		(property "Datasheet" "~"
-			(at 127 166.37 0)
-			(effects
-				(font
-					(size 1.27 1.27)
-				)
-				(hide yes)
-			)
-		)
-		(property "Description" "Generic connector, single row, 01x01, script generated"
-			(at 127 166.37 0)
-			(effects
-				(font
-					(size 1.27 1.27)
-				)
-				(hide yes)
-			)
-		)
-		(pin "1"
-		)
-		(instances
-			(project "mbadge25"
-				(path "/78768b1b-0b2e-4050-96a6-9a18a20b8e29"
-					(reference "J19")
-					(unit 1)
-				)
-			)
-		)
-	)
-	(symbol
 		(lib_id "Library_SYM_mbadge25:Conn_01x01")
 		(at 82.55 21.59 90)
@@
 	)
 	(symbol
-		(lib_id "Library_SYM_mbadge25:Conn_01x01_Pin")
-		(at 127 163.83 180)
-		(unit 1)
-		(exclude_from_sim no)
-		(in_bom no)
-		(on_board yes)
-		(dnp no)
-		(property "Reference" "J18"
-			(at 128.778 163.83 0)
-			(effects
-				(font
-					(size 1.27 1.27)
-				)
-			)
-		)
-		(property "Value" "Conn_IO7.SDA"
-			(at 126.365 161.29 0)
-			(effects
-				(font
-					(size 1.27 1.27)
-				)
-				(hide yes)
-			)
-		)
-		(property "Footprint" "Library_FP_mbadge25:PinHeader_1x01_P1.27mm_Vertical"
-			(at 127 163.83 0)
-			(effects
-				(font
-					(size 1.27 1.27)
-				)
-				(hide yes)
-			)
-		)
-		(property "Datasheet" "~"
-			(at 127 163.83 0)
-			(effects
-				(font
-					(size 1.27 1.27)
-				)
-				(hide yes)
-			)
-		)
-		(property "Description" "Generic connector, single row, 01x01, script generated"
-			(at 127 163.83 0)
-			(effects
-				(font
-					(size 1.27 1.27)
-				)
-				(hide yes)
-			)
-		)
-		(pin "1"
-		)
-		(instances
-			(project "mbadge25"
-				(path "/78768b1b-0b2e-4050-96a6-9a18a20b8e29"
-					(reference "J18")
-					(unit 1)
-				)
-			)
-		)
-	)
-	(symbol
 		(lib_id "Library_SYM_mbadge25:D-Schottky")
 		(at 118.11 39.37 90)
@@
 					(unit 1)
 				)
-			)
-		)
-	)
-	(symbol
-		(lib_id "Library_SYM_mbadge25:Conn_01x01_Pin")
-		(at 127 161.29 180)
-		(unit 1)
-		(exclude_from_sim no)
-		(in_bom no)
-		(on_board yes)
-		(dnp no)
-		(property "Reference" "J17"
-			(at 128.778 161.29 0)
-			(effects
-				(font
-					(size 1.27 1.27)
-				)
-			)
-		)
-		(property "Value" "Conn_IO6.RGB"
-			(at 126.365 158.75 0)
-			(effects
-				(font
-					(size 1.27 1.27)
-				)
-				(hide yes)
-			)
-		)
-		(property "Footprint" "Library_FP_mbadge25:PinHeader_1x01_P1.27mm_Vertical"
-			(at 127 161.29 0)
-			(effects
-				(font
-					(size 1.27 1.27)
-				)
-				(hide yes)
-			)
-		)
-		(property "Datasheet" "~"
-			(at 127 161.29 0)
-			(effects
-				(font
-					(size 1.27 1.27)
-				)
-				(hide yes)
-			)
-		)
-		(property "Description" "Generic connector, single row, 01x01, script generated"
-			(at 127 161.29 0)
-			(effects
-				(font
-					(size 1.27 1.27)
-				)
-				(hide yes)
-			)
-		)
-		(pin "1"
-		)
-		(instances
-			(project "mbadge25"
-				(path "/78768b1b-0b2e-4050-96a6-9a18a20b8e29"
-					(reference "J17")
-					(unit 1)
-				)

Commit message: PCB updates
Parts:
- J24: footprint Library_FP_mbadge25:PinSocket_2x03_P2.54mm_Vertical -> Library_FP_mbadge25:Simple_Addon_v2-BADGE-2x3
Changed lines of the file:
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@@
 	(title_block
 		(title "mbadge25")
-		(date "2025-03-20")
+		(date "2025-03-26")
 		(rev "v1")
 		(company "MakerVille")
-		(comment 1 "minimalistic badge for MakerVille 2025")
+		(comment 2 "URL : badge.makerville.io")
+		(comment 3 "minimalistic badge for MakerVille 2025")
 	)
 	(rectangle
@@
 		)
 	)
+	(image
+		(at 271.78 173.99)
+		(scale 0.519128)
+		(data "iVBORw0KGgoAAAANSUhEUgAAAGQAAABkCAYAAABw4pVUAAAACXBIWXMAAA7DAAAOwwHHb6hkAAAA"
+			"GXRFWHRTb2Z0d2FyZQB3d3cuaW5rc2NhcGUub3Jnm+48GgAADzhJREFUeJztXX2UXVV1//32eZMs"
+			"Mm+SNxNIghVoiGYSQZEiH00JCZEPC/JhsIsPCcZV7Kq1Ii1tY2GtLpbVCsJaSl26qC61GiAFiqjL"
+			"IpBg0CQSpIgUCpmQQBFiSAgzQzITJTN37/5x70zenHffvHffe/fdF2d+a9018/Y995x9zu/eez7u"
+			"PnvTzNDKIDkTQLdzboGZzTezbhGZY2btANoBdEZ/AWAQQB+AQZKDqrqT5FaSW4MgeB7AVjN7I5ua"
+			"VAe2GiEk5zjnFpvZWQDOBjC3wUXsBLCR5LogCB4ys5cbnH9daAlCSC4UkRUALgEwv8nF9wC4T1VX"
+			"m9mWJpddgswIIXm4iFxBcoWZvS8TJTyQ/IWZrVbVNVm92ppOCMmjReTvAfw5gMMSXr6b5PNm9iKA"
+			"AYR9Rn/0PwDkARQQ9il5kvPMbAGAWQnL+S2Ab6jqrWb2SsJr60LTCCH5ThH5DIAVANqquGQ3gPUA"
+			"HlXVpwD0mFl/jWV3ApgvIicCOBPAUlRH0gEA31XVm8xsey1lJ4aZpXoAmCEit4nIsIjYeIdz7nER"
+			"uRbA8YhulpR0IoDjReRvnHO/qKSXiAyJyJcATE+9vdLM3Dl3gYi8UqGyr4rIbQBOSLuy4xC0QERu"
+			"FJHtFXT9jXPuqlRvlpQqOJfk+gqV+5Vz7lIAkhURMXqLc+5SEXl6PN1JrgNwzCFBiHNuuYj0jfNa"
+			"esw598E077IGEEPn3IXRK7QcMb3OuYtalhAAU6O+QstUYGfaj3sah3Puz0TktTJ10uh1O6WlCAFw"
+			"pHPuiTJKD0dKz8i6ceuoX0FEvlJuYOKc2wxgdksQAuCdIvJiGTK2Azg56wZtIDGnjlPXFwAcmykh"
+			"AE4SkV1lOr77AXRm3YgpkDJdRO4uQ8prAE7MhBAAS0Rkb4xSb4nIJ7NuuJRJoYhcIyIHYur/JoDF"
+			"teZd00yd5HtE5KcIlymKMSgiHx4aGnowcaaHINra2t6vqvcD6PBO7VXVM83sl0nzTEwIyXkisgnA"
+			"bO9Ur6p+0MweS6rEoQySJ4vIfwE4wjv1uqqebmZbE+WXhBCSR0Zk+N8ofq2q55hZT5LCf19AsltE"
+			"1gI4yju1LSJlV9V5VUsIyanOuY1WulT+uqounqhkjIDkAhHZAOBwT/54EARnmNmBavKRagsUkVtj"
+			"yNivqhdNdDIAwMy2qOp5OPgpYER+qoh8IUlGFY9okdCfgR/I5XLnZj3iabUjl8u9X0R+58/onXMX"
+			"VzWCq2KId7SIvBEzvPurrCvfqoeIXBu39gVgbl2EAGDcqi3Je7OudCsfUbvdH9NuaytdO26nnsvl"
+			"rjSz1Z54u6qeZGZvVvNKLLDQGTicNfJbA24btL6nqn6nZozp7FpsTueM/D4smPLj3bZ7YLxrAIBk"
+			"QUR+CW9ESvLS4eHhe8peOA7LM0Rkp79QiIRrU9Mw46R2KVjR8VbedV6W9V1czZGXwjXtUgiK9Z+B"
+			"GfMSPCmnxSxIvgqgo9w1ZUdZIvLPAOZ44q+a2ROV7o4KmGJmd+Vd59/WmU9qIMkO13mjAbchwUjU"
+			"h5ltBvB1T/wHInJj2bLjXlmRQcLzAFyR+DVVXVDtq2oE7SycROF/lyn+5oGg9zNJ8ksbJF1eCrcb"
+			"cHXc+ZzaO/qtv2qDB5KdIrIFY40qhlW120LrmTGIZV9C65BiMkDyuqRkVIatyrvOb5PMNTbf2kBy"
+			"6jQW7ilHRi0wsz6SqzxxTkT+IS59CSEkjwZwpSfbHATBmkYp6WFlnoX/JI9KaqPVUHSyszDNFdaR"
+			"WN7ovIMg+A7JJz3xSpJv99OWECKhEdsUT/w5G284VieMuKjdDfy4i10z0ipjPLTziCOHBI/ScHoa"
+			"+Udt93lPPFVE/s5PO4YQkocjtCgsxtNBEDzQWBVjYFhyQGzTNM4suWvSRIGFeZDhDQBOSLOcIAi+"
+			"D+BZT/zxyLp/FGMIEZEr4Jl3kvx8mk+Hh+NEdMN0Tu9uRmHtLLxvWPgYgXlpl2VmRtJf05omIpcV"
+			"C/wn5Mqx6fFyEAT3paHgOPhDFffzaZz5x2kW0tFWWEbhIyj9jpEagiC4G8CrxTKSK4p/S9GJhWZ2"
+			"spfHHWam6alYFl0iujbfNvMDaWTeketcbsoHAExPI/9yMLMAwJ2e7FSSC0Z+jxIi4f6MMVDVO1LV"
+			"cHy0Q/UH+VzX5Y3MtMN1/bUZ7gUwtZH5VgtV/a4vE5GPjP5fJL+kOFG0VyLrDSxTYHZn3hVKRiO1"
+			"IO8Kqwz2FdQx+64XZvZczBB4tO0FAKLx8HzvwrTmHUlBgLfkXedtJFlTBqTrcF3/BvCmRitXC2La"
+			"diHJtwERIc65Zf5Fqrq2CbolwTXtUvj3pLP6aPb9Hwb7i7QUSwpVXefLnHNnAhEhZnamd343gOfS"
+			"Vy0xrmpn4XvVzupncVa+nYUfkfhw2oolxP8A2FMsGOFg5F3qE7K+iXOPZCAuyLt9P5nO6TPHS5bn"
+			"rDn7ZWgDePBbTKsgatv1nngZAEg0UzzGO+knbimY8TQV97Nys/rDWJhrMrQBwHubrFoS+G08l2SX"
+			"AFjgp1TVXzVHp7rwLhHd6M/q8+x6txNuJPCOrBSrBqr6dIx4vjjn4pYpDhWznmOiWf0iAOhg51KI"
+			"bQTwtoz1qgYlUwrnXLeYmU/ILqtxt2tG6KLoQx2u8DkTPIgmz75rhZn1orRj7xYzGzP/IJnh02F3"
+			"Afa7pFcRyBt4A2qYfRswALC80UGKIDnmKbHQj4vM9oQvNVetgyDxQyo/AKDBXybLotdUzjHoT5pU"
+			"3hj4bS0is8XMfFP6ZjVGLPZZ30+pPB3AjpSLelk0WLTf3sjSWn9v8Q8z6xCU7m3Y1zx94rHPep8N"
+			"1BYDeCGlIp5TlcV7bW/Wgxe/rWMJqWgE1gz81vpfgg4tBpB408u4IB8XDZbstzea6sOkDGIJyXvC"
+			"liAEAAZsYNc0bVsC48MNydDwo8HgsGV7be+eyombglhCWhq7bffAoPVd0ICR0OpB619utmN/QxRL"
+			"CYLSJ8J/YjKHmR0Y1L4rCLu9xiz+dVD7P2pmQw1VrH6U9N+C0sem5QgBws+f+4L+TwCWxNLRAFs1"
+			"EPR9ukUXS6sixE/UUhgI+m8m+EkAlb71Dxtx9UDQ/8Vm6FUjSgkh6ROSibFaEuwLer9mxCXjzOr3"
+			"G3nR4HDft5qqWHKMWeYhuU9UdZcnbLQX0FQwONz3fQrPgze5AtAnynMGh3vTN+6rE35bq+ou8deu"
+			"YhYbWxb7hvrWm9oyhF84AeA3UC7Za72bstSrWljoD3IUJLeUEAJgduSj8JDAoPU/6VT/BGYPqMpp"
+			"A9b7TNY6VQOSXSjdQt2TC4KgR6RkOjIfwOPNUq5evGlvbgNwftZ6JETJh8EgCHoEMR+jJPTeOYkU"
+			"ISJxn5e3ioUOg313277RwyQajBhLn5fMrG/kXeV/D1haq1HaJCqDIZZ64keAg5aLvgXELADHpa/a"
+			"hMUJKO3Q1wMRIUEQlHwxE5Gzm6LaBISI+LZiFgTBQULMbAe8zp1kQ63OJzEGfts+b2Y7AaDYTvY+"
+			"ANeP/DCzk0keZ2b/2wQFAQAKthdYaPociMJpTSuLfJeI/JEnHt0UNUqIqn5HRK4vThVtcbshXRUP"
+			"goZvDgu/2azysoCIfNSXqeroJp7RGaGZbSXpe2lYQdJhEg1B1JZXeLLNVuRvbMwU3UodzRzlnGs1"
+			"y/FDFs65ywCMsUf223wMIaq6BmEwk+ILrp+ck9QPkmJm/+iJ96vq3cUC/wnZA8B/h7/HOXdBCjpO"
+			"KDjnPoTSud3XzQutVLKqqKpfRBhZphg3TD4ltYMkzex6T/yWqt7qpy0hxMKYS6s92SnOOX8P+ySq"
+			"hHPuYwD8oe63ovnfGMSaAanqTQCGi2VmdgtJ35P1JCqAZJeZ+ZtNh6I3UQliCTGzbQC+6olnR07N"
+			"JpEAIvIvKPUW8WUz+7/Y9OUyUtV/QhgVsxifIHlqXRpOIJBcBODjnvhVVf1suWvKbjE2s725XO46"
+			"M7urSOxE5B6SJ0YbTiorhSk7gAMt5TWuHhCsKuBk5EnuTpT6k7nWzMqb61Zy5EjykRh3p9/DIRa6"
+			"qJlH2O78YUy7PVjp2oq2vWa2EsCYu4Lkh0TkU9XcKRMRInIdSX/u1mdmf1nx2koJzOwVkisB+KaY"
+			"t+ZyuT+tXs2JgVwudz4A3y+WkfxYuY58bMoqH0MR+VKM++xBAIuyfkW0ygHgFBEZiGmnm6vNI0m4"
+			"iinOuQ1mdop3ak8UriJrz0GZIgpBvgHATE/+8yAIllqVlvdV7w8xswNBEFwIYJt36nAReajYCddE"
+			"Q0TGw/DIALA1CIKLqyUDSOg3ysx2qeq5KJ2fHC0im6Jx94QCyVNE5GfwltUB7FTVc83s9ST5Jd5B"
+			"ZWYvRqT4zgW6ROThXC53XtI8D1W0tbWdLSKPwLMgQRgU7PyqOnEfdXRgZ4hIf0wHdkDCENy/t/MU"
+			"hGHzrpMwrLdf/37UETavXsWOlzD8dlxgyR8A6Mq68VIgYwbJe+PqLCI7kVVgySIFjxWRF8oo+BKA"
+			"07JuxAaSsUhEXi5T1x5UEUEndUIiRWc75zaXUTQQka/hEA7DirB/vD2qS1xw4k0AjmhIWQ1UOici"
+			"N5ZTWsI4Vp9GCwW0r6JOdM5dJWXi/Uqrhu8uPpxzF0p8ELGRu+kJ59zFrdzpAxDn3HIRebJcPURk"
+			"j3Pu/IaXnVKFjiG5dpzKmIg845y7HIDLmoAivZ1z7iMi8ux4upN8CMBRqeiQZgWj+IflOsHRmEzR"
+			"Y//eDIlYGL1uy8VKHzl2OOeuSlOXmqJFJwHJDgljLn0KQFuFtE+a2ZrIZ/AzlpJyJAXAuyW08L8c"
+			"pQYIPoYAfFlVP2vjfVxqhG5pEzJaEHmsiKwCsBKlAWPi8DqARwE8qqpPAeixKr9SxpQ9E0C3iJxo"
+			"ZkujzTL+7DoObwH4tqrebLXMumtA0wgZLZB8u4RRfK4GkNTqfA/JLWa2HaGPlgEAfTjoryUPoDP6"
+			"myc5z8Ktx9U0fjH2A/iGqt5iMaY6aaLphIwWTM4UkctIrjCzljCciAyf71DVNbU+jXXrkBUhY5QI"
+			"45FfiTBKwMImF/8cgPtU9Q5LGIw+DbQEIcUgOds5d4aZnQXgLADHNriInQA2klwXBMGDZvbrBudf"
+			"F1qOEB+RV4lu59wCM+s2s/kiMsfM2hF60yngoEupAYSfBfaRHFDVXSR7SPYEQdCDcGDQl01NqsP/"
+			"A/1Z4dCxv+NhAAAAAElFTkSuQmCCAAAAAAAAAAAAAAAAAAAAAAAAAAAAAAAAAAAAAAAAAAAAAAAA"
+			"AAAAAAAAAAAAAAAAAAAAAAAAAAAAAAAAAAAAAAAAAAAAAAAAAAAAAAAAAAAAAAAAAAAAAAAAAAAA"
+			"AAAAAFUHAACAY6nRjGMAAGA0m9yMYwAAEAAAABAAAAAQAAAAEAAAAAEAAAAAAAAAAAAAAAAAAAAA"
+			"AAAAAAAAALEEAAAAAAAAEPWn3IxjAAAQK6fcjGMAAAAAAAAAAAAAAAAAAAAAAAAAAAAAAAAAAAAA"
+			"AAAAAAAAeNWn3IxjAAAAAAAA/wAAAAEAAAAAAAAAAAAAAAAAAAAAAAAAAAAAAAAAAAAAAAAAAAAA"
+			"AAAAAAAAAAAAAAAAAAAAAAAAAAAAAAAAAAAAAAAAAAAAAAAAAAAAAAAAAAAAAAAAAAAAAAAAAAAA"
+			"AAAAAAAAAAAAAAAAAAAAAAAAAAAAAAAAAAAAAAAAAAAAAAAAAAAAAAAAAAAAAAAAAAAAAAAAAAAA"
+			"AAAAd3d3zx8fHzYAAAAAAAAAAAAAAAAAAAAAAAAAAAAAAAAAAAAAAAAAAAAAAAAAAAAAAAAAAAAA"
+			"AAAAAAAAAAAAACsrK0qFhYXnFhYWJwAAAAAAAAAAAAAAAAAAAAAAAAAAAAAAAAAAAAAAAAAAAAAA"
+			"AAAAAAAAAAAAAAAAAAAAAAAAAAAAOTk5Y39/f90NDQ0XAAAAAAAAAAAAAAAAAAAAAAAAAAAAAAAA"
+			"AAAAAAAAAAAAAAAAAAAAAAAAAAAAAAAAAAAAAAAAAABKSkqAdXV1ywcHBwwAAAAAAAAAAAAAAAAA"
+			"AAAAAAAAAAAAAAAAAAAAAAAAAAAAAAAAAAAAAAAAAAAAAAAAAAAAAQEBAVpaWpxnZ2eyAAAAAAAA"
+			"AAAAAAAAAAAAAAAAAAAAAAAAAAAAAAAAAAAAAAAAAAAAAAAAAAAAAAAAAAAAAAEBAQFaWlqcZ2dn"
+			"sgAAAAAAAAAAAAAAAAAAAAAAAQAAOwEAACkEAAABAAAAAAAAAAAAAAAAAAAA7EiBAn7rdczwxKfc"
+			"jGMAAAAAAAAAAAAAYMpfRp59AAAg319Gnn0AAOxIgQd+63XM7EgjR2ZodMwAAAAAAAAAAAAAAAA6"
+			"Ojpkf39/3Q0NDRcAAAAAAAAAAAAAAAAAAAAAAAAAAAAAAAAAAAAAAAAAAAAAAAAAAAAAAAAAAAAA"
+			"AAArKytKhYWF5xYWFiYAAAAAAAAAAAAAAAAAAAAAAAAAAAAAAAAAAAAAAAAAAAAAAAAAAAAAAAAA"
+			"AAAAAAAAAAAAkQEAAAAAAAAgOwCInn0AACA7AIiefQAAAAAAAAAAAAAAAAAAAAAAAAAAAAAAAAAA"
+			"AAAAAAAAAAAAAAAAAAAAAAAAAA=="
+		)
+	)
 	(label "DP"
 		(at 201.93 55.88 180)
@@
 			)
 		)
-		(property "Footprint" "Library_FP_mbadge25:PinSocket_2x03_P2.54mm_Vertical"
+		(property "Footprint" "Library_FP_mbadge25:Simple_Addon_v2-BADGE-2x3"
 			(at 252.73 50.8 0)
 			(effects
