File: hw_pcb/mbadge25_v1/mbadge25.kicad_pcb (KiCad board)
At the start: 2 copper layers, 46 x 46 mm, 62 parts, among them J1 USB4105-GF-A, J10 Conn_IO20.RX, J11 Conn_IO19.USBP, J12 Conn_IO18.USBN, J15 Conn_IO4, J16 Conn_IO5, J2 BAT, J20 Conn_IO10, J21 Conn_IO00, J22 Conn_IO01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

Commit message: PCB updates
Other:
- board text added: "v1"
Changed lines of the file:
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@@
+		(layer "B.SilkS")
+	)
+	(gr_rect
+		(start 97.5 65.5)
+		(end 102.5 70.5)
+		(stroke
+			(width 0.3)
+			(type solid)
+		)
+		(fill no)
+		(layer "B.SilkS")
+	)
+	(gr_rect
+		(start 81.5 65.5)
+		(end 97.5 70.5)
+		(stroke
+			(width 0.3)
+			(type solid)
+		)
+		(fill yes)
 		(layer "B.SilkS")
 	)
@@
 		(layer "Edge.Cuts")
 	)
+	(gr_text "v1"
+		(at 100 68 0)
+		(layer "B.SilkS")
+		(effects
+			(font
+				(face "Ubuntu Mono")
+				(size 2 2)
+				(thickness 0.4)
+				(bold yes)
+			)
+			(justify mirror)
+		)
+		(render_cache "v1" 0
+			(polygon
+				(pts
+					(xy 100.959507 68.83) (xy 101.149895 68.414298) (xy 101.245326 68.178326) (xy 101.341625 67.917264)
+					(xy 101.432686 67.647265) (xy 101.522243 67.357215) (xy 101.11912 67.357215) (xy 101.023865 67.698789)
+					(xy 100.906262 68.061367) (xy 100.791468 68.382058) (xy 100.703297 68.148196) (xy 100.60389 67.882215)
+					(xy 100.508635 67.609274) (xy 100.435851 67.357215) (xy 100.043841 67.357215) (xy 100.13509 67.646912)
+					(xy 100.231542 67.917264) (xy 100.334553 68.178303) (xy 100.435851 68.414298) (xy 100.634664 68.83)
+				)
+			)
+			(polygon
+				(pts
+					(xy 99.739637 68.83) (xy 99.739637 68.510774) (xy 99.330774 68.510774) (xy 99.330774 67.424382)
+					(xy 99.422359 67.481827) (xy 99.531053 67.535024) (xy 99.722784 67.61196) (xy 99.848813 67.292857)
+					(xy 99.744349 67.248733) (xy 99.626308 67.189298) (xy 99.396597 67.047882) (xy 99.292358 66.967774)
+					(xy 99.210362 66.889612) (xy 98.947191 66.889612) (xy 98.947191 68.510774) (xy 98.560798 68.510774)
+					(xy 98.560798 68.83)
+				)
+			)
+		)
+	)
 	(dimension

Commit message: Fix typo on silksceen
Parts:
- added kibuzzard-67E616D7: G***, kibuzzard-67E616D7, B.Cu at (100.0, 83.5)
